File: _autosave-HPVDTPower.kicad_sch (KiCad schematic)
At the start: 26 parts, among them J4 Conn_01x04_Pin, Q1 PNP, U1 ESP32-S3-MINI-1, U2 MCP1825S, U3 HX711

Commit message: Update _autosave-HPVDTPower.kicad_sch
Connections:
- net LED: now also U1.7 (IO3)
Other:
- note removed: "LED"
Changed lines of the file:
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@@
-		)
-	)
-	(text "LED\n"
-		(exclude_from_sim no)
-		(at 28.956 49.784 0)
-		(effects
-			(font
-				(size 1.27 1.27)
-			)
 		)
 	)
@@
 	(wire
 		(pts
+			(xy 58.42 26.67) (xy 68.58 26.67)
+		)
+		(stroke
+			(width 0)
+			(type default)
+		)
+	)
+	(wire
+		(pts
+			(xy 120.65 60.96) (xy 129.54 60.96)
+		)
+		(stroke
+			(width 0)
+			(type default)
+		)
+	)
+	(wire
+		(pts
+			(xy 120.65 69.85) (xy 120.65 60.96)
+		)
+		(stroke
+			(width 0)
+			(type default)
+		)
+	)
+	(wire
+		(pts
 			(xy 52.07 118.11) (xy 57.15 118.11)
-		)
-		(stroke
-			(width 0)
-			(type default)
-		)
-	)
-	(wire
-		(pts
-			(xy 58.42 26.67) (xy 68.58 26.67)
-		)
-		(stroke
-			(width 0)
-			(type default)
-		)
-	)
-	(wire
-		(pts
-			(xy 120.65 60.96) (xy 129.54 60.96)
-		)
-		(stroke
-			(width 0)
-			(type default)
-		)
-	)
-	(wire
-		(pts
-			(xy 120.65 69.85) (xy 120.65 60.96)
 		)
 		(stroke
@@
 		)
 	)
+	(label "LED"
+		(at 31.75 49.53 0)
+		(effects
+			(font
+				(size 1.27 1.27)
+			)
+			(justify left bottom)
+		)
+	)
 	(label "HX711_{DOUT}"
 		(at 252.73 57.15 0)
@@
 	)
 	(label "LED"
-		(at 52.07 118.11 180)
-		(effects
-			(font
-				(size 1.27 1.27)
-			)
-			(justify right bottom)
-		)
-	)
+		(at 52.07 118.11 0)
+		(effects
+			(font
+				(size 1.27 1.27)
+			)
+			(justify left bottom)
+		)
+	)
